Commit message: fix: update go2w asset to accelerated training

File: source/robot_lab/data/Robots/unitree/go2w_description/urdf/go2w_description.urdf (robot description, URDF)
Before this commit: robot go2w_description, 33 links, 32 joints
Links:
- link FL_calf: geometry collision box size=0.026 0.026 0.12; visual mesh filename=package://go2w_description/meshes/calf.stl
- link FL_calflower: geometry collision box size=0.022 0.022 0.065
- link FL_calflower1: geometry collision box size=0.031 0.031 0.03
- link FL_foot: geometry collision cylinder length=0.045 radius=0.086; visual mesh filename=package://go2w_description/meshes/left_wheel.dae
- link FL_foot_motor: geometry 
- link FL_hip: geometry collision sphere radius=0.046; visual mesh filename=package://go2w_description/meshes/hip.dae
- link FR_calf: geometry collision box size=0.026 0.026 0.12; visual mesh filename=package://go2w_description/meshes/calf_mirror.stl
- link FR_calflower: geometry collision box size=0.022 0.022 0.065
- link FR_calflower1: geometry collision box size=0.031 0.031 0.03
- link FR_foot: geometry collision cylinder length=0.045 radius=0.086; visual mesh filename=package://go2w_description/meshes/right_wheel.dae
- link FR_foot_motor: geometry 
- link FR_hip: geometry collision sphere radius=0.046; visual mesh filename=package://go2w_description/meshes/hip.dae
- link Head_upper: geometry collision sphere radius=0.06
- link RL_calf: geometry collision box size=0.026 0.026 0.12; visual mesh filename=package://go2w_description/meshes/calf.stl
- link RL_calflower: geometry collision box size=0.022 0.022 0.065
- link RL_calflower1: geometry collision box size=0.031 0.031 0.03
- link RL_foot: geometry collision cylinder length=0.045 radius=0.086; visual mesh filename=package://go2w_description/meshes/left_wheel.dae
- link RL_foot_motor: geometry 
- link RL_hip: geometry collision sphere radius=0.046; visual mesh filename=package://go2w_description/meshes/hip.dae
- link RR_calf: geometry collision box size=0.026 0.026 0.12; visual mesh filename=package://go2w_description/meshes/calf_mirror.stl
- link RR_calflower: geometry collision box size=0.022 0.022 0.065
- link RR_calflower1: geometry collision box size=0.031 0.031 0.03
- link RR_foot: geometry collision cylinder length=0.045 radius=0.086; visual mesh filename=package://go2w_description/meshes/right_wheel.dae
- link RR_foot_motor: geometry 
- link RR_hip: geometry collision sphere radius=0.046; visual mesh filename=package://go2w_description/meshes/hip.dae
